File: hardware/STPM32_Breakout/STPM32_Breakout.kicad_pcb (KiCad board)
At the start: 2 copper layers, 38.2 x 28 mm, 34 parts, among them J1 BREADBOARD I/O, SW1 RESET, U1 STPM32, Y1 16MHz

Commit message: Add STPM32 SPI UART mode selector
Co-authored-by: Copilot <223556219+Copilot@users.noreply.github.com>
Parts:
- added SJ1: SPI / UART, SolderJumper-3_P1.3mm_Bridged12_Pad1.0x1.5mm, B.Cu at (54.5, 25.0)
Connections:
- R12 pad 2: DGND -> MODE_BIAS
Routing:
- net MODE_BIAS: track 0.00 -> 29.3 mm, vias 0 -> 1
- net DGND: track 62.4 -> 34.3 mm, vias 0 -> 1
- net +3V3: track 40.4 -> 51.3 mm
Other:
- board text added: "SPI"
- board text added: "UART"
- board text added: "v1.1 2026-10-05"
- board text removed: "v1.0 2026-10-05"
