File: hardware/STPM33_Breakout/STPM33_Breakout.kicad_sch (KiCad schematic)
At the start: 0 parts

Commit message: Build production STPM33 breakout
Implement the dual-current isolated-voltage schematic, routed PCB, sourcing metadata, project-local assets, renders, and ERC/DRC-gated Elecrow fabrication package. Document the SPI/UART selector and reproducible KiCad 10 workflow.

Co-authored-by: Copilot <223556219+Copilot@users.noreply.github.com>
Parts:
- added C1, C2, C3, C4: 330n, Capacitor_SMD:C_0603_1608Metric, symbol Device:C
- added C10, C9: 1u, Capacitor_SMD:C_0805_2012Metric, symbol Device:C
- added C11: 4.7u, Capacitor_SMD:C_0805_2012Metric, symbol Device:C
- added C12, C15: 100n, Capacitor_SMD:C_0603_1608Metric, symbol Device:C
- added C13, C14: 15p, Capacitor_SMD:C_0603_1608Metric, symbol Device:C
- added C5, C6: 33n, Capacitor_SMD:C_0603_1608Metric, symbol Device:C
- added J1: BREADBOARD I/O, Connector_PinHeader_2.54mm:PinHeader_1x14_P2.54mm_Vertical, symbol Connector_Generic:Conn_01x14
- added NT1: ANALOG/DIGITAL STAR, NetTie:NetTie-3_SMD_Pad0.5mm, symbol Connector_Generic:Conn_01x03
- added R1, R2, R3, R4: 100R, Resistor_SMD:R_0603_1608Metric, symbol Device:R
- added R10, R7: 2.49k, Resistor_SMD:R_0603_1608Metric, symbol Device:R
- added R11, R12: 1k, Resistor_SMD:R_0603_1608Metric, symbol Device:R
- added R13, R14: 10k, Resistor_SMD:R_0603_1608Metric, symbol Device:R
- added R5, R6, R8, R9: 100k, Resistor_SMD:R_0603_1608Metric, symbol Device:R
- added RB1, RB2: 2.4R, Resistor_SMD:R_0603_1608Metric, symbol Device:R
- added SJ1: SPI / UART, Jumper:SolderJumper-3_P1.3mm_Bridged12_Pad1.0x1.5mm, symbol Connector_Generic:Conn_01x03
- added SW1: RESET, Button_Switch_SMD:SW_SPST_CK_RS282G05A3, symbol Switch:SW_Push
- added TP1: INT1, TestPoint:TestPoint_Pad_D1.5mm, symbol Connector_Generic:Conn_01x01
- added TP2: INT2, TestPoint:TestPoint_Pad_D1.5mm, symbol Connector_Generic:Conn_01x01
- added TP3: LED1, TestPoint:TestPoint_Pad_D1.5mm, symbol Connector_Generic:Conn_01x01
- added TP4: LED2, TestPoint:TestPoint_Pad_D1.5mm, symbol Connector_Generic:Conn_01x01
- added TP5: CLKOUT_ZCR, TestPoint:TestPoint_Pad_D1.5mm, symbol Connector_Generic:Conn_01x01
- added U1: STPM33, Package_DFN_QFN:QFN-32-1EP_5x5mm_P0.5mm_EP3.45x3.45mm, symbol STPM3x:STPM33
- added Y1: 16MHz, Crystal:Crystal_SMD_3225-4Pin_3.2x2.5mm, symbol Device:Crystal
Connections:
- new net +3V3: C9.1, J1.1 (Pin_1), R13.1, SJ1.3 (Pin_3), U1.23 (VCC)
- new net CLKOUT_ZCR: TP5.1 (Pin_1), U1.1 (CLKOUT/ZCR)
- new net CT1_N: J1.6 (Pin_6), R2.1, RB1.2
- new net CT1_P: J1.5 (Pin_5), R1.1, RB1.1
- new net CT2_N: J1.8 (Pin_8), R4.1, RB2.2
- new net CT2_P: J1.7 (Pin_7), R3.1, RB2.1
- new net DGND: C11.2, C13.2, C14.2, C9.2, J1.2 (Pin_2), NT1.3 (Pin_3), SJ1.1 (Pin_1), SW1.2, U1.26 (GNDD)
- new net EN: J1.14 (Pin_14), R13.2, SW1.1, U1.8 (EN)
- new net GNDA: C1.2, C10.2, C2.2, C3.2, C4.2, C5.2, C6.2, NT1.1 (Pin_1), R10.2, R7.2, U1.20 (GNDA), U1.22 (GND_REG)
- new net GND_REF: C12.2, C15.2, NT1.2 (Pin_2), U1.18 (GND_REF)
- new net IIN1: C2.1, R2.2, U1.12 (IIN1)
- new net IIN2: C4.1, R4.2, U1.13 (IIN2)
- new net IIP1: C1.1, R1.2, U1.11 (IIP1)
- new net IIP2: C3.1, R3.2, U1.14 (IIP2)
- new net INT1: TP1.1 (Pin_1), U1.6 (INT1)
- new net INT2: TP2.1 (Pin_1), U1.7 (INT2)
- new net LED1: TP3.1 (Pin_1), U1.4 (LED1)
- new net LED2: TP4.1 (Pin_1), U1.5 (LED2)
- new net MISO_TXD: J1.12 (Pin_12), U1.32 (MISO/TXD)
- new net MODE_BIAS: R14.2, SJ1.2 (Pin_2)
- new net MOSI_RXD: J1.11 (Pin_11), U1.31 (MOSI/RXD)
- new net SCL: J1.10 (Pin_10), U1.30 (SCL)
- new net SCS: J1.9 (Pin_9), R14.1, U1.29 (SCS)
- new net SYN: J1.13 (Pin_13), U1.28 (SYN)
- new net VAC_N: J1.4 (Pin_4), R8.1
- new net VAC_N_MID: R8.2, R9.1
- new net VAC_P: J1.3 (Pin_3), R5.1
- new net VAC_P_MID: R5.2, R6.1
- new net VDDA: C10.1, U1.21 (VDDA)
- new net VDDD: C11.1, U1.27 (VDDD)
- new net VDIV_N: R10.1, R12.1, R9.2
- new net VDIV_P: R11.1, R6.2, R7.1
- new net VIN1: C6.1, R12.2, U1.10 (VIN1)
- new net VIP1: C5.1, R11.2, U1.9 (VIP1)
- new net VREF1: C12.1, U1.17 (VREF1)
- new net VREF2: C15.1, U1.19 (VREF2)
- new net XTAL1: C13.1, U1.3 (XTAL1), Y1.1
- new net XTAL2: C14.1, U1.2 (CLKIN/XTAL2), Y1.2
- no-connect marks 0 -> 4
Other:
- note added: "STPM33 supports SPI or UART; I2C is not supported. SJ1 1-2 closed = SPI default. Cut 1-2 and bridge 2-3 for UART."
- note added: "TWO CURRENT HEADER INPUTS: 100 A : 50 mA current-output CTs Each channel: 2.4 ohm burden = 120 mV RMS at 100 A; approx. 4.8 kHz LPF."
- note added: "VOLTAGE HEADER INPUT: isolated 9 VAC transformer secondary only 200k/2.49k symmetric divider = approx. 111 mV RMS differential at 9 VAC."
- note added: "WARNING: NOT A CERTIFIED ISOLATION BARRIER. Never connect J1 directly to mains."
- title: STPM33 Breakout -> STPM33 Energy Metering Breakout
